File: SSUAV.kicad_sch (KiCad schematic)
At the start: 15 parts, among them U2 LM2596S-11V

Commit message: Add files via upload
Parts:
- added XT-60_Power_Module1: ~, symbol AESC:XT-60
Connections:
- net +BATT: now also XT-60_Power_Module1.1 (Vin)
- net GND: now also XT-60_Power_Module1.2 (GND)
